File: shield/BrewPi Shield.sch (EAGLE design)
At the start: 31 parts, among them J1 ARDUINO_R3_SHIELD_ICSP, U1 SN74HC595N, U2 P-CHANNEL-MOSFET

Commit message: Version 1.2 upload
Parts:
- removed D1, D2: 1N4004, diode:1N4004
- removed U2: P-CHANNEL-MOSFET, GeekAmmo:P-CHANNEL-MOSFET
- added Q1: 2N3906, transistor-pnp:2N3906
- added R12: 10k Ohm, SparkFun-Passives:RESISTORAXIAL-0.3
- R10: value 20-30 -> 220; device SparkFun-Passives:RESISTORPTH-1/2W -> SparkFun-Passives:RESISTORAXIAL-0.3
- R11: value 220 -> 150 Ohm
- RELAY: value 555 -> (none)
Connections:
- removed net N$10: LCD.15, R10.1
- removed net N$11: D1.A, U2.D
- removed net N$9: D2.C, R10.2
- new net N$7: Q1.C, R11.1
- net 5V: now also BTOOTH.4, Q1.E, R10.2; no longer BTOOTH.3, R11.2
- net A5V: no longer U2.S
- net GND: now also BTOOTH.3; no longer BTOOTH.4
- net N$13: now also R10.1; no longer R11.1
- net N$2: now also Q1.B, R12.2; no longer U1.QC, U2.G
- net N$3: now also BTOOTH.1; no longer BTOOTH.2
- net N$5: now also LCD.15, R11.2; no longer D1.C, D2.A
- net QB: now also R12.1
- net RX: now also BTOOTH.2; no longer BTOOTH.1
Other:
- moved on the sheet: R10, R11

Commit message: Version 1.3 upload
Parts:
- removed BTOOTH: (no value), con-lstb:MA04-1
- removed LCD: 16 pin, pinhead:PINHD-1X16
- removed LEDS: (no value), pinhead:PINHD-1X2
- added ALARM, DOOR: 2 pin, LBussy:HEADER02-1
- added COOL_LED, HEAT_LED, ONE_WIRE_SEL: 3 pin, LBussy:HEADER03-1
- added I2C_LED, ROT_ENC, SERIAL: 4 pin, LBussy:HEADER04-1
- added PARALLEL_LCD_1, PARALLEL_LCD_2: 6 pin, LBussy:HEADER06-1
- added R13*: 10kΩ, SparkFun-Passives:RESISTORAXIAL-0.3
- added RJ45: RJ45-8X, con-tycoelectronics:RJ45-8X
- C1, C2, C3, C4: value .1UF -> 0.1μF
- C5, C6, C7: value (none) -> 0.1μF
- C8: value 1.0UF -> 1.0μF
- PROBE1, PROBE2, PROBE3: value (none) -> 3 pin; device con-lstb:MA03-1 -> LBussy:HEADER03-1
- R1, R3, R4, R5: value 10K -> 10kΩ
- R10, R9: value 220 -> 220Ω
- R11: value 150 Ohm -> 150Ω
- R12: value 10k Ohm -> 10kΩ
- R2: value 0-20K -> 20kΩ
- R6: value 4.7K -> 4.7kΩ
- R7: value 1K -> 2kΩ
- R8: value 2K -> 1kΩ
- RELAY: value (none) -> 4 pin; device con-lstb:MA04-1 -> LBussy:HEADER04-1
Connections:
- removed net 5V: BTOOTH.4, C1.1, C2.1, J1.5V, LCD.2, PROBE1.2, PROBE2.2, PROBE3.2, Q1.E, R1.A, R10.2, R3.2, R4.2, R5.2, R6.1, R9.2, RELAY.3
- removed net A5V: C3.1, C4.1, C8.1, J1.5V@ICSP, R2.2, U1.VCC
- removed net AGND: C3.2, C4.2, C8.2, J1.GND@ICSP, U1.GND, U1.~OE
- removed net D5: J1.*D5, RELAY.2
- removed net D6: J1.*D6, RELAY.1
- removed net D7: C5.1, J1.D7, R3.1
- removed net IO8: C6.1, J1.D8, R4.1
- removed net IO9: C7.1, J1.*D9, R5.1
- removed net N$12: LEDS.1, R9.1
- removed net N$13: LEDS.2, R10.1
- new net 1WIRE: ONE_WIRE_SEL.2, PROBE1.3, PROBE2.3, PROBE3.3, R6.2, RJ45.4
- new net A0: J1.A0, ONE_WIRE_SEL.3
- new net A4: I2C_LED.3, J1.A4, ONE_WIRE_SEL.1
- new net A5: I2C_LED.4, J1.A5
- new net ALARM: ALARM.1, J1.*D3
- new net COOL: J1.*D5, R9.1, RELAY.2, RJ45.7
- new net DOOR: DOOR.1, J1.D4, RJ45.6
- new net HEAT: J1.*D6, R10.2, RELAY.3, RJ45.8
- new net N$8: HEAT_LED.2, R10.1
- new net PSHB: C6.1, J1.D7, R4.1, ROT_ENC.2
- new net QC: R12.1, U1.QC
- new net ROTA: C5.1, J1.*D9, R3.1, ROT_ENC.1
- new net ROTB: C7.1, J1.D8, R5.1, ROT_ENC.4
- new net VCC: C1.1, C2.1, C3.1, C4.1, C8.1, COOL_LED.1, HEAT_LED.1, I2C_LED.2, J1.5V, J1.5V@ICSP, PARALLEL_LCD_1.2, PROBE1.2, PROBE2.2, PROBE3.2, Q1.E, R1.A, R2.2, R3.2, R4.2, R5.2, R6.1, RELAY.4, RJ45.3, SERIAL.4, U1.VCC
- net GND: now also ALARM.2, C3.2, C4.2, C8.2, COOL_LED.3, DOOR.2, HEAT_LED.3, I2C_LED.1, J1.GND@ICSP, PARALLEL_LCD_1.1, PARALLEL_LCD_1.5, PARALLEL_LCD_2.6, R13*.1, R7.1, RELAY.1, RJ45.5, ROT_ENC.3, SERIAL.3, U1.GND, U1.~OE; no longer BTOOTH.3, LCD.1, LCD.16, LCD.5, R8.1, RELAY.4
- net N$2: now also R13*.2
- net N$3: now also R7.2, R8.1, SERIAL.1; no longer BTOOTH.1, R7.1, R8.2
- net N$4: now also COOL_LED.2, R9.2; no longer J1.A4, PROBE1.3, PROBE2.3, PROBE3.3, R6.2
- net N$5: now also PARALLEL_LCD_2.5; no longer LCD.15
- net N$6: now also PARALLEL_LCD_1.3; no longer LCD.3
- net QA: now also PARALLEL_LCD_1.4; no longer LCD.4
- net QB: now also PARALLEL_LCD_1.6; no longer LCD.6, R12.1
- net QE: now also PARALLEL_LCD_2.1; no longer LCD.11
- net QF: now also PARALLEL_LCD_2.2; no longer LCD.12
- net QG: now also PARALLEL_LCD_2.3; no longer LCD.13
- net QH: now also PARALLEL_LCD_2.4; no longer LCD.14
- net RX: now also SERIAL.2; no longer BTOOTH.2
- net TX: now also R8.2; no longer R7.2
Other:
- moved on the sheet: C1, C2, C3, C4, C5, C6, C7, C8, R1, R10, R11, R12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

Commit message: Version 1.3.1 upload
Parts:
- removed R13*: 10kΩ, SparkFun-Passives:RESISTORAXIAL-0.3
- added BACKLIGHT: 3 pin, LBussy:HEADER03-1
Connections:
- new net N$9: Q1.B, R12.2
- net GND: now also BACKLIGHT.1; no longer R13*.1
- net N$2: now also BACKLIGHT.2, R12.1; no longer Q1.B, R12.2, R13*.2
- net QC: now also BACKLIGHT.3; no longer R12.1
Other:
- moved on the sheet: R12
Changed lines of the file:
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@@
 <?xml version="1.0" encoding="utf-8"?>
 <!DOCTYPE eagle SYSTEM "eagle.dtd">
-<eagle version="9.4.1">
+<eagle version="9.4.2">
 <drawing>
 <settings>
@@
 <part name="PARALLEL_LCD_1" library="LBussy" deviceset="HEADER06-1" device="" package3d_urn="urn:adsk.eagle:package:8340/1" value="6 pin"/>
 <part name="ALARM" library="LBussy" deviceset="HEADER02-1" device="" package3d_urn="urn:adsk.eagle:package:22435/2" value="2 pin"/>
-<part name="R13*" library="SparkFun-Passives" deviceset="RESISTOR" device="AXIAL-0.3" value="10kΩ"/>
+<part name="BACKLIGHT" library="LBussy" deviceset="HEADER03-1" device="" package3d_urn="urn:adsk.eagle:package:8339/1" value="3 pin"/>
 </parts>
 <sheets>
@@
 <attribute name="VALUE" x="26.67" y="45.212" size="1.778" layer="96" rot="R180"/>
 </instance>
-<instance part="R12" gate="G$1" x="58.42" y="30.48" smashed="yes" rot="R90">
-<attribute name="NAME" x="56.4134" y="29.21" size="1.778" layer="95" rot="R90"/>
-<attribute name="VALUE" x="61.976" y="28.448" size="1.778" layer="96" rot="R90"/>
-</instance>
-<instance part="Q1" gate="G$1" x="58.42" y="39.37" smashed="yes" rot="MR90">
-<attribute name="VALUE" x="53.34" y="44.45" size="1.778" layer="96" rot="MR180"/>
+<instance part="R12" gate="G$1" x="68.58" y="27.94" smashed="yes" rot="R90">
+<attribute name="NAME" x="66.5734" y="26.67" size="1.778" layer="95" rot="R90"/>
+<attribute name="VALUE" x="72.136" y="25.908" size="1.778" layer="96" rot="R90"/>
+</instance>
+<instance part="Q1" gate="G$1" x="68.58" y="39.37" smashed="yes" rot="MR90">
+<attribute name="VALUE" x="63.5" y="44.45" size="1.778" layer="96" rot="MR180"/>
 </instance>
 <instance part="ONE_WIRE_SEL" gate="G$1" x="55.88" y="-2.54" smashed="yes">
@@
 <attribute name="VALUE" x="80.01" y="-48.26" size="1.778" layer="96"/>
 </instance>
-<instance part="R13*" gate="G$1" x="68.58" y="36.83" smashed="yes" rot="R180">
-<attribute name="NAME" x="72.39" y="35.3314" size="1.778" layer="95" rot="R180"/>
-<attribute name="VALUE" x="72.39" y="40.132" size="1.778" layer="96" rot="R180"/>
+<instance part="BACKLIGHT" gate="G$1" x="68.58" y="12.7" smashed="yes" rot="R90">
+<attribute name="VALUE" x="72.39" y="10.668" size="1.778" layer="96" rot="R180"/>
+<attribute name="NAME" x="75.438" y="21.59" size="1.778" layer="95" rot="R180"/>
 </instance>
 </instances>
@@
 <wire x1="43.18" y1="48.26" x2="58.42" y2="48.26" width="0.1524" layer="91"/>
 <pinref part="C8" gate="G$1" pin="2"/>
-<wire x1="58.42" y1="48.26" x2="119.38" y2="48.26" width="0.1524" layer="91"/>
+<wire x1="58.42" y1="48.26" x2="81.28" y2="48.26" width="0.1524" layer="91"/>
 <junction x="58.42" y="48.26"/>
+<wire x1="81.28" y1="48.26" x2="119.38" y2="48.26" width="0.1524" layer="91"/>
 <wire x1="33.02" y1="48.26" x2="43.18" y2="48.26" width="0.1524" layer="91"/>
 <junction x="33.02" y="48.26"/>
 <junction x="43.18" y="48.26"/>
+<pinref part="BACKLIGHT" gate="G$1" pin="1"/>
+<wire x1="71.12" y1="20.32" x2="71.12" y2="22.86" width="0.1524" layer="91"/>
+<wire x1="71.12" y1="22.86" x2="81.28" y2="22.86" width="0.1524" layer="91"/>
+<wire x1="81.28" y1="22.86" x2="81.28" y2="48.26" width="0.1524" layer="91"/>
+<junction x="81.28" y="48.26"/>
 </segment>
 <segment>
@@
 <wire x1="83.82" y1="-43.18" x2="78.74" y2="-43.18" width="0.1524" layer="91"/>
 <label x="73.66" y="-43.18" size="1.778" layer="95"/>
-</segment>
-<segment>
-<pinref part="R13*" gate="G$1" pin="1"/>
-<wire x1="73.66" y1="36.83" x2="76.2" y2="36.83" width="0.1524" layer="91"/>
-<label x="73.406" y="36.83" size="1.778" layer="95"/>
 </segment>
 </net>
@@
 <segment>
 <pinref part="Q1" gate="G$1" pin="C"/>
-<wire x1="53.34" y1="41.91" x2="27.94" y2="41.91" width="0.1524" layer="91"/>
+<wire x1="63.5" y1="41.91" x2="27.94" y2="41.91" width="0.1524" layer="91"/>
 <pinref part="R11" gate="G$1" pin="1"/>
 </segment>
@@
 </segment>
 <segment>
-<wire x1="-12.7" y1="55.88" x2="5.08" y2="55.88" width="0.1524" layer="91"/>
+<pinref part="U1" gate="A" pin="VCC"/>
+<wire x1="15.24" y1="27.94" x2="12.7" y2="27.94" width="0.1524" layer="91"/>
+<label x="10.16" y="27.94" size="1.778" layer="95"/>
+</segment>
+<segment>
+<pinref part="J1" gate="G$1" pin="5V@ICSP"/>
+<wire x1="91.44" y1="2.54" x2="86.36" y2="2.54" width="0.1524" layer="91"/>
+<label x="86.36" y="2.54" size="1.778" layer="95"/>
+</segment>
+<segment>
+<pinref part="R2" gate="G$1" pin="2"/>
+<wire x1="-12.7" y1="55.88" x2="0" y2="55.88" width="0.1524" layer="91"/>
+<wire x1="0" y1="55.88" x2="5.08" y2="55.88" width="0.1524" layer="91"/>
 <wire x1="5.08" y1="55.88" x2="12.7" y2="55.88" width="0.1524" layer="91"/>
 <pinref part="C2" gate="G$1" pin="1"/>
@@
 <pinref part="C4" gate="G$1" pin="1"/>
 <pinref part="C8" gate="G$1" pin="1"/>
-<wire x1="58.42" y1="55.88" x2="119.38" y2="55.88" width="0.1524" layer="91"/>
+<wire x1="58.42" y1="55.88" x2="76.2" y2="55.88" width="0.1524" layer="91"/>
 <junction x="58.42" y="55.88"/>
+<wire x1="76.2" y1="55.88" x2="119.38" y2="55.88" width="0.1524" layer="91"/>
 <wire x1="33.02" y1="55.88" x2="43.18" y2="55.88" width="0.1524" layer="91"/>
 <junction x="33.02" y="55.88"/>
 <junction x="43.18" y="55.88"/>
-</segment>
-<segment>
+<wire x1="0" y1="33.02" x2="0" y2="55.88" width="0.1524" layer="91"/>
+<junction x="0" y="55.88"/>
 <pinref part="Q1" gate="G$1" pin="E"/>
-<wire x1="63.5" y1="41.91" x2="68.834" y2="41.91" width="0.1524" layer="91"/>
-<label x="65.532" y="42.164" size="1.778" layer="95"/>
-</segment>
-<segment>
-<pinref part="U1" gate="A" pin="VCC"/>
-<wire x1="15.24" y1="27.94" x2="12.7" y2="27.94" width="0.1524" layer="91"/>
-<label x="10.16" y="27.94" size="1.778" layer="95"/>
-</segment>
-<segment>
-<pinref part="J1" gate="G$1" pin="5V@ICSP"/>
-<wire x1="91.44" y1="2.54" x2="86.36" y2="2.54" width="0.1524" layer="91"/>
-<label x="86.36" y="2.54" size="1.778" layer="95"/>
-</segment>
-<segment>
-<pinref part="R2" gate="G$1" pin="2"/>
-<wire x1="0" y1="33.02" x2="0" y2="38.1" width="0.1524" layer="91"/>
-<label x="0" y="38.1" size="1.778" layer="95"/>
+<wire x1="76.2" y1="55.88" x2="76.2" y2="41.91" width="0.1524" layer="91"/>
+<wire x1="76.2" y1="41.91" x2="73.66" y2="41.91" width="0.1524" layer="91"/>
+<junction x="76.2" y="55.88"/>
 </segment>
 <segment>
@@
 </segment>
 </net>
+<net name="QC" class="0">
+<segment>
+<pinref part="U1" gate="A" pin="QC"/>
+<label x="50.8" y="22.86" size="1.778" layer="95"/>
+<pinref part="BACKLIGHT" gate="G$1" pin="3"/>
+<wire x1="66.04" y1="20.32" x2="66.04" y2="22.86" width="0.1524" layer="91"/>
+<wire x1="66.04" y1="22.86" x2="50.8" y2="22.86" width="0.1524" layer="91"/>
+</segment>
+</net>
 <net name="N$2" class="0">
 <segment>
+<pinref part="BACKLIGHT" gate="G$1" pin="2"/>
+<pinref part="R12" gate="G$1" pin="1"/>
+<wire x1="68.58" y1="20.32" x2="68.58" y2="22.86" width="0.1524" layer="91"/>
+</segment>
+</net>
+<net name="N$9" class="0">
+<segment>
+<pinref part="R12" gate="G$1" pin="2"/>
 <pinref part="Q1" gate="G$1" pin="B"/>
-<pinref part="R12" gate="G$1" pin="2"/>
-<wire x1="58.42" y1="36.83" x2="58.42" y2="35.56" width="0.1524" layer="91"/>
-<wire x1="58.42" y1="36.83" x2="63.5" y2="36.83" width="0.1524" layer="91"/>
-<junction x="58.42" y="36.83"/>
-<pinref part="R13*" gate="G$1" pin="2"/>
-</segment>
-</net>
-<net name="QC" class="0">
-<segment>
-<pinref part="U1" gate="A" pin="QC"/>
-<wire x1="50.8" y1="22.86" x2="58.42" y2="22.86" width="0.1524" layer="91"/>
-<pinref part="R12" gate="G$1" pin="1"/>
-<wire x1="58.42" y1="22.86" x2="58.42" y2="25.4" width="0.1524" layer="91"/>
-<label x="50.8" y="22.86" size="1.778" layer="95"/>
-</segment>
-</net>
+<wire x1="68.58" y1="33.02" x2="68.58" y2="36.83" width="0.1524" layer="91"/>
+</segment>
+</net>
