File: Uno Shield/BrewPi Shield.brd (EAGLE design)
At the start: 53.6 x 59.7 mm, 39 parts, among them J1 ARDUINO_R3_SHIELD_ICSP, Q1 2N3906, U1 SN74HC595N

Commit message: Add RJ45 Breakout
Routing:
- net GND: track 274.3 -> 290.6 mm
- net A0: track 18.6 -> 22.9 mm
- net VCC: track 235.8 -> 239.4 mm
- net A5: track 59.6 -> 61.3 mm, vias 2 -> 0
- net QC: track 25.3 -> 26.8 mm
- net A4: track 62.9 -> 64.0 mm
- net N$6: track 20.0 -> 21.1 mm
- net COOL: track 78.2 -> 79.3 mm
- net N$5: track 8.40 -> 9.44 mm
- net RX: track 11.0 -> 12.0 mm
- net QA: track 28.9 -> 29.9 mm
- net ALARM: track 17.0 -> 18.0 mm
- net ROTA: track 22.7 -> 23.6 mm
- net ROTB: track 23.7 -> 24.3 mm
- net 1WIRE: track 62.0 -> 62.6 mm
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