File: Uno Shield/Combo Shield/BrewPi Combo Shield.brd (EAGLE design)
At the start: 53.6 x 59.7 mm, 39 parts, among them J1 ARDUINO_R3_SHIELD_ICSP, Q1 2N3906, U1 SN74HC595N

Commit message: Add voltage select header
Other:
- board text added: "BrewPi Remix I2C/RevC Shield v1.3.3 by @LBussy Based on a design by @day_trippr"
- board text removed: "BrewPi Remix I2C/RevC Shield @CadiBrewer v1.3.1a Inspired by @LBussy Based on a design by @day_trippr"
Changed lines of the file:
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@@
 <?xml version="1.0" encoding="utf-8"?>
 <!DOCTYPE eagle SYSTEM "eagle.dtd">
-<eagle version="9.5.2">
+<eagle version="9.6.2">
 <drawing>
 <settings>
-<setting alwaysvectorfont="yes"/>
+<setting alwaysvectorfont="no"/>
 <setting keepoldvectorfont="yes"/>
 <setting verticaltext="up"/>
@@
 <text x="63.1" y="61.2" size="0.8128" layer="25" font="vector" ratio="10">GND</text>
 <text x="72.1614" y="51.3207" size="0.8128" layer="26" font="vector" ratio="10" rot="MR0">BrewPi Remix I2C/RevC Shield
-@CadiBrewer v1.3.1a
-Inspired by @LBussy
+v1.3.3 by @LBussy
 Based on a design by @day_trippr</text>
 <text x="72.1614" y="39.9288" size="0.8128" layer="26" font="vector" rot="MR0">RJ45 Pinout:
